Commit message: 把原本的2D雷达转化为3D雷达，使他适配Fast_LIO

File: src/smartcar_description/urdf/xacro/smartcar_body.xacro (robot description, xacro)
@@ -4,5 +4,6 @@
   	<!-- Macro for SmartCar body. Including Gazebo extensions, but does not include Kinect -->
   	<include filename="$(find smartcar_description)/urdf/xacro/smartcar_sim.xacro"/>
-	<xacro:include filename="$(find smartcar_description)/urdf/xacro/sensors/lidar.xacro" />
+	<!-- <xacro:include filename="$(find smartcar_description)/urdf/xacro/sensors/lidar.xacro" /> -->
+    <xacro:include filename="$(find velodyne_description)/urdf/VLP-16.urdf.xacro"/>
 	<xacro:include filename="$(find smartcar_description)/urdf/xacro/sensors/imu.xacro" />
 	<xacro:include filename="$(find smartcar_description)/urdf/xacro/rm_description/urdf/RML63/rml_63.xacro" />
@@ -415,4 +416,5 @@
 		</joint>
 	<!--	Sensors-->
+        <!--
 		<xacro:lidar prefix="laser_front"/>
 		<joint name="lidar_front_joint" type="fixed">
@@ -427,4 +429,8 @@
 			<child link="laser_back_link"/>
 		</joint>
+        -->
+        <xacro:VLP-16 parent="base_link" name="velodyne" topic="/velodyne_points" hz="10" samples="440" gpu="false">
+            <origin xyz="0 0 0.4" rpy="0 0 0" />
+        </xacro:VLP-16>
 		<xacro:imu prefix="imu"/>
 		<joint name="imu_joint" type="fixed">

Commit message: 去掉机械臂，方便跑通算法

File: src/smartcar_description/urdf/xacro/smartcar_body.xacro (robot description, xacro)
@@ -7,5 +7,4 @@
     <xacro:include filename="$(find velodyne_description)/urdf/VLP-16.urdf.xacro"/>
 	<xacro:include filename="$(find smartcar_description)/urdf/xacro/sensors/imu.xacro" />
-	<xacro:include filename="$(find smartcar_description)/urdf/xacro/rm_description/urdf/RML63/rml_63.xacro" />
   	<xacro:macro name="smartcar_body">
 		<xacro:property name="wheel_m" value="2.0"/>
@@ -146,31 +145,4 @@
 			</collision>
 		</link>
-		<joint name="arm_slider_joint" type="prismatic">
-			<axis xyz="0 0 1"/>
-			<origin xyz="0.2 0 0" rpy="0 0 0" />
-			<parent link="column_link"/>
-			<child link="arm_slider_link" />
-			<dynamics damping="0.1"/>
-			<limit effort="100" velocity="0.1" lower="-0.4" upper="0.4" />
-			<joint_properties damping="20.0" friction="100.0"/>
-		</joint>
-		<link name="arm_slider_link">
-			<xacro:cube_inertial_matrix m="0.1" a="0.1" b="0.2" c="0.1" />
-			<visual>
-				<origin xyz="0 0 0" rpy="0 0 0" />
-				<geometry>
-					<box size="0.1 0.2 0.1"/>
-				</geometry>
-				<material name="gray">
-					<color rgba="0.5 0.5 0.5 1"/>
-				</material>
-			</visual>
-			<collision>
-				<origin xyz="0 0 0" rpy="0 0 0" />
-				<geometry>
-					<box size="0.1 0.2 0.1" />
-				</geometry>
-			</collision>
-		</link>
 		<link name="left_front_wheel">
 			<xacro:cylinder_inertial_matrix m="${wheel_m}" r="${wheel_r}" h="${wheel_h}"/>
@@ -439,18 +411,4 @@
 			<child link="imu_link"/>
 		</joint>
-		<xacro:rml_63 prefix="left"/>
-		<joint name="arm_left_joint" type="fixed">
-			<axis xyz="0 1 0"/>
-			<origin xyz="0 0.1 0" rpy="${-M_PI/2} 0 0" />
-			<parent link="arm_slider_link"/>
-			<child link="rml_link_left" />
-		</joint>
-		<xacro:rml_63 prefix="right"/>
-		<joint name="arm_right_joint" type="fixed">
-			<axis xyz="0 1 0"/>
-			<origin xyz="0 -0.1 0" rpy="${M_PI/2} 0 0" />
-			<parent link="arm_slider_link"/>
-			<child link="rml_link_right" />
-		</joint>
 	</xacro:macro>
 </robot>

File: src/smartcar_description/urdf/xacro/smartcar_sim.xacro (robot description, xacro)
@@ -59,7 +59,4 @@
 		</gazebo>
 		<gazebo reference="column_link">
-			<material>Gazebo/Gray</material>
-		</gazebo>
-		<gazebo reference="arm_slider_link">
 			<material>Gazebo/Gray</material>
 		</gazebo>
@@ -136,5 +133,4 @@
 <!--		<xacro:transmission_effort joint_name="arm_left_joint"/>-->
 <!--		<xacro:transmission_effort joint_name="arm_right_joint"/>-->
-		<xacro:transmission_position joint_name="arm_slider_joint"/>
 <!--		<xacro:transmission_position joint_name="arm_left_joint"/>-->
 <!--		<xacro:transmission_position joint_name="arm_right_joint"/>-->
